Commit message: update files

File: model/urdf/york_base.urdf (robot description, URDF)
Before this commit: robot york_urdf, 9 links, 8 joints
Links:
- link base_link: geometry collision mesh filename=package://york_joy_control/model/meshes/base_link.STL; visual mesh filename=package://york_joy_control/model/meshes/base_link.STL
- link blw_Link: geometry collision mesh filename=package://york_joy_control/model/meshes/blw_Link.STL; visual mesh filename=package://york_joy_control/model/meshes/blw_Link.STL
- link brw_Link: geometry collision mesh filename=package://york_joy_control/model/meshes/brw_Link.STL; visual mesh filename=package://york_joy_control/model/meshes/brw_Link.STL
- link fb_Link: geometry collision mesh filename=package://york_joy_control/model/meshes/fb_Link.STL; visual mesh filename=package://york_joy_control/model/meshes/fb_Link.STL
- link flw_Link: geometry collision mesh filename=package://york_joy_control/model/meshes/flw_Link.STL; visual mesh filename=package://york_joy_control/model/meshes/flw_Link.STL
- link frw_Link: geometry collision mesh filename=package://york_joy_control/model/meshes/frw_Link.STL; visual mesh filename=package://york_joy_control/model/meshes/frw_Link.STL
- link p_Link: geometry collision mesh filename=package://york_joy_control/model/meshes/p_Link.STL; visual mesh filename=package://york_joy_control/model/meshes/p_Link.STL
- link print_Link: geometry collision mesh filename=package://york_joy_control/model/meshes/print_Link.STL; visual mesh filename=package://york_joy_control/model/meshes/print_Link.STL
- link up_Link: geometry collision mesh filename=package://york_joy_control/model/meshes/up_Link.STL; visual mesh filename=package://york_joy_control/model/meshes/up_Link.STL
